File: MCU.kicad_sch (KiCad schematic)
At the start: 7 parts, among them U1 STM32G0B1KBT6, X1 8MHz SX2M8.000M20F30TNN

Commit message: Fix the stale exposed-pad notes; document the JLC panel and CAN limit
MCU sheet: the LQFP-32 has no exposed pad, so drop the QFN-era paste
window / thermal via note and the hidden-pin label text. Schematic PDF
re-exported.

README: the card is panelised by JLC on the order (fingers on an outer
edge, mouse-bites, no V-cut), and CAN must never share a cable with
more than 12 V (accepted for Rev A).
Other:
- note added: "1. U1 STM32G0B1KBT6 — LQFP-32 (0.8 mm), non-N pinout (PA9/PA10 on 19/21, PA11/PA12 on 22/23). Order exactly STM32G0B1KBT6, NOT the …KBT6N variant (pins 17, 20, 26–29 differ; VDDIO2 on pin 20). Footprint: KiCad LQFP-32_7x7mm_P0.8mm (IPC), checked against the DS13560 LQFP32 drawing. No exposed pad: pin 5 is the only VSS pin. 2. Decoupling (ST AN5096): C4 100 nF + C5 10 µF 0805 (≈ 6.9 µF at 3.3 V) a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"
- note added: "LQFP-32: no exposed pad; pin 5 is the only VSS. Pin 5 runs to the C4/C5 ground pads and the GND plane."
- note removed: "1. U1 STM32G0B1KBT6 — LQFP-32 (0.8 mm), non-N pinout (PA9/PA10 on 19/21, PA11/PA12 on 22/23). Order exactly STM32G0B1KBT6, NOT the …KBT6N variant (pins 17, 20, 26–29 differ; VDDIO2 on pin 20). Footprint: KiCad LQFP-32_7x7mm_P0.8mm (IPC), checked against the DS13560 LQFP32 drawing. Exposed pad = VSS: 2×2 paste windows + 5 thermal vias (0.5/0.25 mm) to the GND plane. 2. Decoupling (ST AN5096): C4 1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"
- note removed: "LQFP-32: no exposed pad; pin 5 is the only VSS. Hidden in the symbol, stacked behind pin 5. Soldered to GND with 5 vias (see pin table)."
Changed lines of the file:
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@@
 		)
 	)
-	(text "LQFP-32: no exposed pad; pin 5 is the only VSS.\nHidden in the symbol, stacked behind pin 5.\nSoldered to GND with 5 vias (see pin table)."
+	(text "LQFP-32: no exposed pad; pin 5 is the only VSS.\nPin 5 runs to the C4/C5 ground pads and the GND plane."
 		(exclude_from_sim no)
 		(at 128.524 108.966 0)
@@
 		)
 	)
-	(text "1. U1 STM32G0B1KBT6 — LQFP-32 (0.8 mm), non-N pinout (PA9/PA10 on 19/21, PA11/PA12 on 22/23).\n   Order exactly STM32G0B1KBT6, NOT the …KBT6N variant (pins 17, 20, 26–29 differ; VDDIO2 on pin 20).\n   Footprint: KiCad LQFP-32_7x7mm_P0.8mm (IPC), checked against the DS13560 LQFP32 drawing.\n   Exposed pad = VSS: 2×2 paste windows + 5 thermal vias (0.5/0.25 mm) to the GND plane.\n\n2. Decoupling (ST AN5096): C4 100 nF + C5 10 µF 0805 (≈ 6.9 µF at 3.3 V) at VDD pin 4.\n   C6 100 nF on NRST (internal pull-up ≈ 40 kΩ) filters reset glitches.\n\n3. Clock tree\n   X1 8 MHz CMOS XO (±20 + ±30 ppm, duty 45–55 %, OE high) → R14 22 Ω → PC14 (HSE bypass).\n   32-pin package: PC14 = only HSE input, no OSC_OUT (PC15 OSC_EN = optional AF; GPIO here) → no crystal.\n   PLL:  input = 8 MHz / M(2) = 4 MHz (50 % duty; PLL needs 45–55 %)   VCO = 4 MHz × N(32) = 128 MHz\n         SYSCLK = VCO / R(2) = 64 MHz        FDCAN kernel = VCO / Q(2) = 64 MHz\n   HSE line X1 → R14 → PC14: ≤ 8 mm, no vias, 0.3 mm spacing; R14 22 Ω at X1 OUT (less ringing/EMI).\n\n4. CAN bit timing — FDCAN2, 500 kbit/s classic (CANopen)\n   f_bit = 64 MHz / (BRP 8 × (1 + TSEG1 13 + TSEG2 2)) = 64 MHz / 128 = 500 kbit/s\n   Sample point = (1 + 13) / 16 = 87.5 % (CANopen recommendation), SJW = 2\n   Oscillator ≈ ±53 ppm worst ≪ CAN limit 0.485 % OK   (HSI16 drifts −2.75/+2.0 %: not usable for CAN)\n\n5. Pin allocation\n   PB0 / PB1 ..... FDCAN2 RX / TX → U3          PB4 / PB5 ... CAN_LED / USER_LED\n   PA9 / PA10 .... USART1 TX / RX → ST-Link VCP PB7 ........ BUZZER (TIM4_CH2 PWM)\n   PA11 / PA12 ... USB DN / DP (wired, unused)  PB2 ........ VSENSE_5V (ADC1_IN10, ÷3)\n   PA13 / PA14 ... SWDIO / SWCLK(BOOT0)         PB8 / PB9 .. I2C1 SCL / SDA (carrier monitors)\n   PF2 ........... NRST                         PC14 ....... HSE_IN\n   To carrier (14 GPIO): PA0–PA8, PA15, PB3, PB6, PC6, PC15  (ADC-capable: PA0–PA7)\n\n6. Boot, programming & debug\n   PA14 = SWCLK and BOOT0. Option bytes: nBOOT_SEL = 1, nBOOT0 = 1 (check/set once in STM32CubeProgrammer)\n   → always boots from flash; the PA14 pin is NOT read as BOOT0 → SWCLK stays free and a\n     connected debugger can never change the boot mode.\n   No BOOT0 button (it would fight the ST-Link's SWCLK driver). Flash/debug = ST-Link over SWD.\n   A blank chip starts the ST bootloader; after the first SWD flash, power-cycle once (the\n     empty-flash flag is only re-read at power-on).\n   ST bootloader when needed: firmware jumps to system memory on a VCP command,\n     or clear nBOOT0 via SWD → use the bootloader → set nBOOT0 = 1 again.\n   ST system bootloader (AN2606): USART1 PA9/PA10 (8E1, via ST-Link VCP). It also probes USART2\n     PA2/PA3, SPI1 PA4–PA7, USB PA11/PA12 and I2C1 PB6/PB7 (pulled up: PB6 = no gate drive).\n   No FDCAN bootloader on this package (needs PD0/PD1).\n   VCP default: USART1 115200 8N1 → ST-Link V3MINIE (STDC14 pins 13/14).\n\n7. Monitoring (firmware)\n   VDDA = 3.0 V × VREFINT_CAL / VREFINT_DATA  (factory calibration at 3.0 V)\n   V(+5V) = ADC(PB2) / 4095 × VDDA × 3   (R8 20k / R9 10k)\n   Unused GPIO → analog mode (lowest power, best EMC)."
+	(text "1. U1 STM32G0B1KBT6 — LQFP-32 (0.8 mm), non-N pinout (PA9/PA10 on 19/21, PA11/PA12 on 22/23).\n   Order exactly STM32G0B1KBT6, NOT the …KBT6N variant (pins 17, 20, 26–29 differ; VDDIO2 on pin 20).\n   Footprint: KiCad LQFP-32_7x7mm_P0.8mm (IPC), checked against the DS13560 LQFP32 drawing.\n   No exposed pad: pin 5 is the only VSS pin.\n\n2. Decoupling (ST AN5096): C4 100 nF + C5 10 µF 0805 (≈ 6.9 µF at 3.3 V) at VDD pin 4.\n   C6 100 nF on NRST (internal pull-up ≈ 40 kΩ) filters reset glitches.\n\n3. Clock tree\n   X1 8 MHz CMOS XO (±20 + ±30 ppm, duty 45–55 %, OE high) → R14 22 Ω → PC14 (HSE bypass).\n   32-pin package: PC14 = only HSE input, no OSC_OUT (PC15 OSC_EN = optional AF; GPIO here) → no crystal.\n   PLL:  input = 8 MHz / M(2) = 4 MHz (50 % duty; PLL needs 45–55 %)   VCO = 4 MHz × N(32) = 128 MHz\n         SYSCLK = VCO / R(2) = 64 MHz        FDCAN kernel = VCO / Q(2) = 64 MHz\n   HSE line X1 → R14 → PC14: ≤ 8 mm, no vias, 0.3 mm spacing; R14 22 Ω at X1 OUT (less ringing/EMI).\n\n4. CAN bit timing — FDCAN2, 500 kbit/s classic (CANopen)\n   f_bit = 64 MHz / (BRP 8 × (1 + TSEG1 13 + TSEG2 2)) = 64 MHz / 128 = 500 kbit/s\n   Sample point = (1 + 13) / 16 = 87.5 % (CANopen recommendation), SJW = 2\n   Oscillator ≈ ±53 ppm worst ≪ CAN limit 0.485 % OK   (HSI16 drifts −2.75/+2.0 %: not usable for CAN)\n\n5. Pin allocation\n   PB0 / PB1 ..... FDCAN2 RX / TX → U3          PB4 / PB5 ... CAN_LED / USER_LED\n   PA9 / PA10 .... USART1 TX / RX → ST-Link VCP PB7 ........ BUZZER (TIM4_CH2 PWM)\n   PA11 / PA12 ... USB DN / DP (wired, unused)  PB2 ........ VSENSE_5V (ADC1_IN10, ÷3)\n   PA13 / PA14 ... SWDIO / SWCLK(BOOT0)         PB8 / PB9 .. I2C1 SCL / SDA (carrier monitors)\n   PF2 ........... NRST                         PC14 ....... HSE_IN\n   To carrier (14 GPIO): PA0–PA8, PA15, PB3, PB6, PC6, PC15  (ADC-capable: PA0–PA7)\n\n6. Boot, programming & debug\n   PA14 = SWCLK and BOOT0. Option bytes: nBOOT_SEL = 1, nBOOT0 = 1 (check/set once in STM32CubeProgrammer)\n   → always boots from flash; the PA14 pin is NOT read as BOOT0 → SWCLK stays free and a\n     connected debugger can never change the boot mode.\n   No BOOT0 button (it would fight the ST-Link's SWCLK driver). Flash/debug = ST-Link over SWD.\n   A blank chip starts the ST bootloader; after the first SWD flash, power-cycle once (the\n     empty-flash flag is only re-read at power-on).\n   ST bootloader when needed: firmware jumps to system memory on a VCP command,\n     or clear nBOOT0 via SWD → use the bootloader → set nBOOT0 = 1 again.\n   ST system bootloader (AN2606): USART1 PA9/PA10 (8E1, via ST-Link VCP). It also probes USART2\n     PA2/PA3, SPI1 PA4–PA7, USB PA11/PA12 and I2C1 PB6/PB7 (pulled up: PB6 = no gate drive).\n   No FDCAN bootloader on this package (needs PD0/PD1).\n   VCP default: USART1 115200 8N1 → ST-Link V3MINIE (STDC14 pins 13/14).\n\n7. Monitoring (firmware)\n   VDDA = 3.0 V × VREFINT_CAL / VREFINT_DATA  (factory calibration at 3.0 V)\n   V(+5V) = ADC(PB2) / 4095 × VDDA × 3   (R8 20k / R9 10k)\n   Unused GPIO → analog mode (lowest power, best EMC)."
 		(exclude_from_sim no)
 		(at 281.94 33.02 0)
